Commit message: fix: prevent Foxglove wheel geometry overscaling

File: robot/description/robot.urdf (robot description, URDF)
Before this commit: robot robot, 10 links, 9 joints
Links:
- link left_wheel: geometry collision sphere radius=0.033; visual box size=0.066 0.026 0.066
- link right_wheel: geometry collision sphere radius=0.033; visual box size=0.066 0.026 0.066

File: robot/description/robot_core.xacro (robot description, xacro)
@@ -76,7 +76,9 @@
         <visual>
             <geometry>
-                <cylinder radius="${wheel_radius}" length="${wheel_thickness}"/>
+                <!-- Foxglove Web can over-scale rotating cylinder primitives.
+                     A box keeps the same physical footprint without covering the map. -->
+                <box size="${wheel_radius * 2} ${wheel_thickness} ${wheel_radius * 2}"/>
             </geometry>
-            <material name="blue"/>
+            <material name="black"/>
         </visual>
         <collision>
@@ -99,7 +101,7 @@
         <visual>
             <geometry>
-                <cylinder radius="${wheel_radius}" length="${wheel_thickness}"/>
+                <box size="${wheel_radius * 2} ${wheel_thickness} ${wheel_radius * 2}"/>
             </geometry>
-            <material name="blue"/>
+            <material name="black"/>
         </visual>
         <collision>

Commit message: fix: remove oversized sphere primitives from Foxglove model

File: robot/description/robot.urdf (robot description, URDF)
Before this commit: robot robot, 10 links, 9 joints
Links:
- link caster_wheel: geometry collision box size=0.02 0.02 0.02; visual box size=0.02 0.02 0.02
- link left_wheel: geometry collision box size=0.066 0.026 0.066; visual box size=0.066 0.026 0.066
- link right_wheel: geometry collision box size=0.066 0.026 0.066; visual box size=0.066 0.026 0.066

File: robot/description/robot_core.xacro (robot description, xacro)
@@ -84,5 +84,5 @@
         <collision>
             <geometry>
-                <sphere radius="${wheel_radius}"/>
+                <box size="${wheel_radius * 2} ${wheel_thickness} ${wheel_radius * 2}"/>
             </geometry>
         </collision>
@@ -107,5 +107,5 @@
         <collision>
             <geometry>
-                <sphere radius="${wheel_radius}"/>
+                <box size="${wheel_radius * 2} ${wheel_thickness} ${wheel_radius * 2}"/>
             </geometry>
         </collision>
@@ -123,5 +123,5 @@
         <visual>
             <geometry>
-                <sphere radius="${caster_wheel_radius}"/>
+                <box size="${caster_wheel_radius * 2} ${caster_wheel_radius * 2} ${caster_wheel_radius * 2}"/>
             </geometry>
             <material name="white"/>
@@ -129,5 +129,5 @@
         <collision>
             <geometry>
-                <sphere radius="${caster_wheel_radius}"/>
+                <box size="${caster_wheel_radius * 2} ${caster_wheel_radius * 2} ${caster_wheel_radius * 2}"/>
             </geometry>
         </collision>
