Commit message: fix(slam): update 4-wheel kinematics, center lidar at base_link, and calibrate scan matcher

File: robot/description/lidar.xacro (robot description, xacro)
@@ -2,7 +2,7 @@
 <robot xmlns:xacro="http://www.ros.org/wiki/xacro" >
     <joint name="laser_joint" type="fixed">
-        <parent link="chassis"/>
+        <parent link="base_link"/>
         <child link="laser_frame"/>
-        <origin xyz="0.122 0 0.212" rpy="0 0 0"/>
+        <origin xyz="0 0 0.16" rpy="0 0 0"/>
     </joint>
     <link name="laser_frame">

File: robot/description/robot.urdf (robot description, URDF)
Before this commit: robot robot, 10 links, 9 joints
Links:
- removed link caster_wheel
- added link front_left_wheel, mass 0.05; collision sphere radius=0.033; visual cylinder length=0.026 radius=0.033
- added link front_right_wheel, mass 0.05; collision sphere radius=0.033; visual cylinder length=0.026 radius=0.033
- added link rear_left_wheel, mass 0.05; collision sphere radius=0.033; visual cylinder length=0.026 radius=0.033
- added link rear_right_wheel, mass 0.05; collision sphere radius=0.033; visual cylinder length=0.026 radius=0.033
- link chassis: mass 0.5 -> 1.0; geometry collision box size=0.28 0.20 0.10; visual box size=0.28 0.20 0.10
- link left_wheel: mass 0.05 -> None; geometry 
- link right_wheel: mass 0.05 -> None; geometry 
Joints:
- removed joint caster_wheel_joint
- added joint front_left_wheel_joint: type continuous, parent base_link, child front_left_wheel, origin xyz=0.08 0.11 0 rpy=-1.5707963267948966 0 0, axis 0 0 1
- added joint front_right_wheel_joint: type continuous, parent base_link, child front_right_wheel, origin xyz=0.08 -0.11 0 rpy=1.5707963267948966 0 0, axis 0 0 -1
- added joint rear_left_wheel_joint: type continuous, parent base_link, child rear_left_wheel, origin xyz=-0.08 0.11 0 rpy=-1.5707963267948966 0 0, axis 0 0 1
- added joint rear_right_wheel_joint: type continuous, parent base_link, child rear_right_wheel, origin xyz=-0.08 -0.11 0 rpy=1.5707963267948966 0 0, axis 0 0 -1
- joint camera_joint: origin xyz=0.276 0 0.181 rpy=0 0.18 0 -> xyz=0.14 0 0.06 rpy=0 0.18 0
- joint chassis_joint: origin xyz=-0.226 0 -0.01 -> xyz=0 0 0.05 rpy=0 0 0
- joint face_joint: origin xyz=0.335 0 0.069 rpy=0 0 0 -> xyz=0.14 0 0.02 rpy=0 0 0
- joint laser_joint: origin xyz=0.122 0 0.212 rpy=0 0 0 -> xyz=0.0 0.0 0.16 rpy=0 0 0; parent chassis -> base_link
- joint left_wheel_joint: origin xyz=0 0.1485 0 rpy=-1.5707963267948966 0 0 -> xyz=0 0.11 0 rpy=-1.5707963267948966 0 0
- joint right_wheel_joint: origin xyz=0 -0.1485 0 rpy=1.5707963267948966 0 0 -> xyz=0 -0.11 0 rpy=1.5707963267948966 0 0

File: robot/description/robot_core.xacro (robot description, xacro)
@@ -2,18 +2,14 @@
 <robot xmlns:xacro="http://www.ros.org/wiki/xacro" >
     <xacro:include filename="inertial_macros.xacro"/>
-    <xacro:property name="chassis_length" value="0.335"/>
-    <xacro:property name="chassis_width" value="0.265"/>
-    <xacro:property name="chassis_height" value="0.138"/>
+    <xacro:property name="chassis_length" value="0.28"/>
+    <xacro:property name="chassis_width" value="0.20"/>
+    <xacro:property name="chassis_height" value="0.10"/>
     <xacro:property name="chassis_mass" value="1.0"/>
     <xacro:property name="wheel_radius" value="0.033"/>
     <xacro:property name="wheel_thickness" value="0.026"/>
     <xacro:property name="wheel_mass" value="0.05"/>
-    <xacro:property name="wheel_offset_x" value="0.226"/>
-    <xacro:property name="wheel_offset_y" value="0.1485"/>
-    <xacro:property name="wheel_offset_z" value="0.01"/>
-    <xacro:property name="caster_wheel_radius" value="0.01"/>
-    <xacro:property name="caster_wheel_mass" value="0.01"/>
-    <xacro:property name="caster_wheel_offset_x" value="0.075"/>
-    <xacro:property name="caster_wheel_offset_z" value="${wheel_offset_z - wheel_radius + caster_wheel_radius}"/>
+    <xacro:property name="wheel_offset_x" value="0.08"/>
+    <xacro:property name="wheel_offset_y" value="0.11"/>
+    <xacro:property name="wheel_offset_z" value="0.0"/>
     <material name="white">
         <color rgba="1 1 1 1" />
@@ -42,13 +38,13 @@
     <link name="base_footprint">
     </link>
-    <!-- CHASSIS LINK -->
+    <!-- CHASSIS LINK (CENTERED AT BASE_LINK) -->
     <joint name="chassis_joint" type="fixed">
         <parent link="base_link"/>
         <child link="chassis"/>
-        <origin xyz="${-wheel_offset_x} 0 ${-wheel_offset_z}"/>
+        <origin xyz="0 0 0.05"/>
     </joint>
     <link name="chassis">
         <visual>
-            <origin xyz="${chassis_length/2} 0 ${chassis_height/2}"/>
+            <origin xyz="0 0 0"/>
             <geometry>
                 <box size="${chassis_length} ${chassis_width} ${chassis_height}"/>
@@ -57,5 +53,5 @@
         </visual>
         <collision>
-            <origin xyz="${chassis_length/2} 0 ${chassis_height/2}"/>
+            <origin xyz="0 0 0"/>
             <geometry>
                 <box size="${chassis_length} ${chassis_width} ${chassis_height}"/>
@@ -63,15 +59,15 @@
         </collision>
         <xacro:inertial_box mass="0.5" x="${chassis_length}" y="${chassis_width}" z="${chassis_height}">
-            <origin xyz="${chassis_length/2} 0 ${chassis_height/2}" rpy="0 0 0"/>
+            <origin xyz="0 0 0" rpy="0 0 0"/>
         </xacro:inertial_box>
     </link>
-    <!-- LEFT WHEEL LINK -->
-    <joint name="left_wheel_joint" type="continuous">
+    <!-- FRONT LEFT WHEEL (M1) -->
+    <joint name="front_left_wheel_joint" type="continuous">
         <parent link="base_link"/>
-        <child link="left_wheel"/>
-        <origin xyz="0 ${wheel_offset_y} 0" rpy="-${pi/2} 0 0" />
+        <child link="front_left_wheel"/>
+        <origin xyz="${wheel_offset_x} ${wheel_offset_y} 0" rpy="-${pi/2} 0 0" />
         <axis xyz="0 0 1"/>
     </joint>
-    <link name="left_wheel">
+    <link name="front_left_wheel">
         <visual>
             <geometry>
@@ -89,12 +85,12 @@
         </xacro:inertial_cylinder>
     </link>
-    <!-- RIGHT WHEEL LINK -->
-    <joint name="right_wheel_joint" type="continuous">
+    <!-- REAR LEFT WHEEL (M2) -->
+    <joint name="rear_left_wheel_joint" type="continuous">
         <parent link="base_link"/>
-        <child link="right_wheel"/>
-        <origin xyz="0 ${-wheel_offset_y} 0" rpy="${pi/2} 0 0" />
-        <axis xyz="0 0 -1"/>
+        <child link="rear_left_wheel"/>
+        <origin xyz="${-wheel_offset_x} ${wheel_offset_y} 0" rpy="-${pi/2} 0 0" />
+        <axis xyz="0 0 1"/>
     </joint>
-    <link name="right_wheel">
+    <link name="rear_left_wheel">
         <visual>
             <geometry>
@@ -112,29 +108,64 @@
         </xacro:inertial_cylinder>
     </link>
-    <!-- CASTER WHEEL LINK -->
-    <joint name="caster_wheel_joint" type="fixed">
-        <parent link="chassis"/>
-        <child link="caster_wheel"/>
-        <origin xyz="${caster_wheel_offset_x} 0 ${caster_wheel_offset_z}"/>
+    <!-- FRONT RIGHT WHEEL (M3) -->
+    <joint name="front_right_wheel_joint" type="continuous">
+        <parent link="base_link"/>
+        <child link="front_right_wheel"/>
+        <origin xyz="${wheel_offset_x} ${-wheel_offset_y} 0" rpy="${pi/2} 0 0" />
+        <axis xyz="0 0 -1"/>
     </joint>
-    <link name="caster_wheel">
+    <link name="front_right_wheel">
         <visual>
             <geometry>
-                <sphere radius="${caster_wheel_radius}"/>
+                <cylinder radius="${wheel_radius}" length="${wheel_thickness}"/>
             </geometry>
-            <material name="white"/>
+            <material name="blue"/>
         </visual>
         <collision>
             <geometry>
-                <sphere radius="${caster_wheel_radius}"/>
+                <sphere radius="${wheel_radius}"/>
             </geometry>
         </collision>
-        <xacro:inertial_sphere mass="${caster_wheel_mass}" radius="${caster_wheel_radius}">
+        <xacro:inertial_cylinder mass="${wheel_mass}" length="${wheel_thickness}" radius="${wheel_radius}">
             <origin xyz="0 0 0" rpy="0 0 0"/>
-        </xacro:inertial_sphere>
+        </xacro:inertial_cylinder>
     </link>
-    <gazebo reference="caster_wheel">
-        <mu1 value="0.001"/>
-        <mu2 value="0.001"/>
-    </gazebo>
+    <!-- REAR RIGHT WHEEL (M4) -->
+    <joint name="rear_right_wheel_joint" type="continuous">
+        <parent link="base_link"/>
+        <child link="rear_right_wheel"/>
+        <origin xyz="${-wheel_offset_x} ${-wheel_offset_y} 0" rpy="${pi/2} 0 0" />
+        <axis xyz="0 0 -1"/>
+    </joint>
+    <link name="rear_right_wheel">
+        <visual>
+            <geometry>
+                <cylinder radius="${wheel_radius}" length="${wheel_thickness}"/>
+            </geometry>
+            <material name="blue"/>
+        </visual>
+        <collision>
+            <geometry>
+                <sphere radius="${wheel_radius}"/>
+            </geometry>
+        </collision>
+        <xacro:inertial_cylinder mass="${wheel_mass}" length="${wheel_thickness}" radius="${wheel_radius}">
+            <origin xyz="0 0 0" rpy="0 0 0"/>
+        </xacro:inertial_cylinder>
+    </link>
+    <!-- ALIAS MID-WHEEL JOINTS FOR 2WD / DIFF-DRIVE COMPATIBILITY -->
+    <joint name="left_wheel_joint" type="continuous">
+        <parent link="base_link"/>
+        <child link="left_wheel"/>
+        <origin xyz="0 ${wheel_offset_y} 0" rpy="-${pi/2} 0 0" />
+        <axis xyz="0 0 1"/>
+    </joint>
+    <link name="left_wheel"/>
+    <joint name="right_wheel_joint" type="continuous">
+        <parent link="base_link"/>
+        <child link="right_wheel"/>
+        <origin xyz="0 ${-wheel_offset_y} 0" rpy="${pi/2} 0 0" />
+        <axis xyz="0 0 -1"/>
+    </joint>
+    <link name="right_wheel"/>
 </robot>

Commit message: revert: revert autonomous navigation and lidar scan mapping to commit 2a61ed5

File: robot/description/lidar.xacro (robot description, xacro)
@@ -2,7 +2,7 @@
 <robot xmlns:xacro="http://www.ros.org/wiki/xacro" >
     <joint name="laser_joint" type="fixed">
-        <parent link="base_link"/>
+        <parent link="chassis"/>
         <child link="laser_frame"/>
-        <origin xyz="0 0 0.16" rpy="0 0 0"/>
+        <origin xyz="0.122 0 0.212" rpy="0 0 0"/>
     </joint>
     <link name="laser_frame">

File: robot/description/robot.urdf (robot description, URDF)
Before this commit: robot robot, 13 links, 12 joints
Links:
- removed link front_left_wheel
- removed link front_right_wheel
- removed link rear_left_wheel
- removed link rear_right_wheel
- added link caster_wheel, mass 0.01; collision sphere radius=0.01; visual sphere radius=0.01
- link chassis: mass 1.0 -> 0.5; geometry collision box size=0.335 0.265 0.138; visual box size=0.335 0.265 0.138
- link left_wheel: mass None -> 0.05; geometry collision sphere radius=0.033; visual cylinder length=0.026 radius=0.033
- link right_wheel: mass None -> 0.05; geometry collision sphere radius=0.033; visual cylinder length=0.026 radius=0.033
Joints:
- removed joint front_left_wheel_joint
- removed joint front_right_wheel_joint
- removed joint rear_left_wheel_joint
- removed joint rear_right_wheel_joint
- added joint caster_wheel_joint: type fixed, parent chassis, child caster_wheel, origin xyz=0.075 0 -0.013
- joint camera_joint: origin xyz=0.14 0 0.06 rpy=0 0.18 0 -> xyz=0.276 0 0.181 rpy=0 0.18 0
- joint chassis_joint: origin xyz=0 0 0.05 rpy=0 0 0 -> xyz=-0.226 0 -0.01
- joint face_joint: origin xyz=0.14 0 0.02 rpy=0 0 0 -> xyz=0.335 0 0.069 rpy=0 0 0
- joint laser_joint: origin xyz=0.0 0.0 0.16 rpy=0 0 0 -> xyz=0.122 0 0.212 rpy=0 0 0; parent base_link -> chassis
- joint left_wheel_joint: origin xyz=0 0.11 0 rpy=-1.5707963267948966 0 0 -> xyz=0 0.1485 0 rpy=-1.5707963267948966 0 0
- joint right_wheel_joint: origin xyz=0 -0.11 0 rpy=1.5707963267948966 0 0 -> xyz=0 -0.1485 0 rpy=1.5707963267948966 0 0

File: robot/description/robot_core.xacro (robot description, xacro)
@@ -2,14 +2,18 @@
 <robot xmlns:xacro="http://www.ros.org/wiki/xacro" >
     <xacro:include filename="inertial_macros.xacro"/>
-    <xacro:property name="chassis_length" value="0.28"/>
-    <xacro:property name="chassis_width" value="0.20"/>
-    <xacro:property name="chassis_height" value="0.10"/>
+    <xacro:property name="chassis_length" value="0.335"/>
+    <xacro:property name="chassis_width" value="0.265"/>
+    <xacro:property name="chassis_height" value="0.138"/>
     <xacro:property name="chassis_mass" value="1.0"/>
     <xacro:property name="wheel_radius" value="0.033"/>
     <xacro:property name="wheel_thickness" value="0.026"/>
     <xacro:property name="wheel_mass" value="0.05"/>
-    <xacro:property name="wheel_offset_x" value="0.08"/>
-    <xacro:property name="wheel_offset_y" value="0.11"/>
-    <xacro:property name="wheel_offset_z" value="0.0"/>
+    <xacro:property name="wheel_offset_x" value="0.226"/>
+    <xacro:property name="wheel_offset_y" value="0.1485"/>
+    <xacro:property name="wheel_offset_z" value="0.01"/>
+    <xacro:property name="caster_wheel_radius" value="0.01"/>
+    <xacro:property name="caster_wheel_mass" value="0.01"/>
+    <xacro:property name="caster_wheel_offset_x" value="0.075"/>
+    <xacro:property name="caster_wheel_offset_z" value="${wheel_offset_z - wheel_radius + caster_wheel_radius}"/>
     <material name="white">
         <color rgba="1 1 1 1" />
@@ -38,13 +42,13 @@
     <link name="base_footprint">
     </link>
-    <!-- CHASSIS LINK (CENTERED AT BASE_LINK) -->
+    <!-- CHASSIS LINK -->
     <joint name="chassis_joint" type="fixed">
         <parent link="base_link"/>
         <child link="chassis"/>
-        <origin xyz="0 0 0.05"/>
+        <origin xyz="${-wheel_offset_x} 0 ${-wheel_offset_z}"/>
     </joint>
     <link name="chassis">
         <visual>
-            <origin xyz="0 0 0"/>
+            <origin xyz="${chassis_length/2} 0 ${chassis_height/2}"/>
             <geometry>
                 <box size="${chassis_length} ${chassis_width} ${chassis_height}"/>
@@ -53,5 +57,5 @@
         </visual>
         <collision>
-            <origin xyz="0 0 0"/>
+            <origin xyz="${chassis_length/2} 0 ${chassis_height/2}"/>
             <geometry>
                 <box size="${chassis_length} ${chassis_width} ${chassis_height}"/>
@@ -59,15 +63,15 @@
         </collision>
         <xacro:inertial_box mass="0.5" x="${chassis_length}" y="${chassis_width}" z="${chassis_height}">
-            <origin xyz="0 0 0" rpy="0 0 0"/>
+            <origin xyz="${chassis_length/2} 0 ${chassis_height/2}" rpy="0 0 0"/>
         </xacro:inertial_box>
     </link>
-    <!-- FRONT LEFT WHEEL (M1) -->
-    <joint name="front_left_wheel_joint" type="continuous">
+    <!-- LEFT WHEEL LINK -->
+    <joint name="left_wheel_joint" type="continuous">
         <parent link="base_link"/>
-        <child link="front_left_wheel"/>
-        <origin xyz="${wheel_offset_x} ${wheel_offset_y} 0" rpy="-${pi/2} 0 0" />
+        <child link="left_wheel"/>
+        <origin xyz="0 ${wheel_offset_y} 0" rpy="-${pi/2} 0 0" />
         <axis xyz="0 0 1"/>
     </joint>
-    <link name="front_left_wheel">
+    <link name="left_wheel">
         <visual>
             <geometry>
@@ -85,12 +89,12 @@
         </xacro:inertial_cylinder>
     </link>
-    <!-- REAR LEFT WHEEL (M2) -->
-    <joint name="rear_left_wheel_joint" type="continuous">
+    <!-- RIGHT WHEEL LINK -->
+    <joint name="right_wheel_joint" type="continuous">
         <parent link="base_link"/>
-        <child link="rear_left_wheel"/>
-        <origin xyz="${-wheel_offset_x} ${wheel_offset_y} 0" rpy="-${pi/2} 0 0" />
-        <axis xyz="0 0 1"/>
+        <child link="right_wheel"/>
+        <origin xyz="0 ${-wheel_offset_y} 0" rpy="${pi/2} 0 0" />
+        <axis xyz="0 0 -1"/>
     </joint>
-    <link name="rear_left_wheel">
+    <link name="right_wheel">
         <visual>
             <geometry>
@@ -108,64 +112,29 @@
         </xacro:inertial_cylinder>
     </link>
-    <!-- FRONT RIGHT WHEEL (M3) -->
-    <joint name="front_right_wheel_joint" type="continuous">
-        <parent link="base_link"/>
-        <child link="front_right_wheel"/>
-        <origin xyz="${wheel_offset_x} ${-wheel_offset_y} 0" rpy="${pi/2} 0 0" />
-        <axis xyz="0 0 -1"/>
+    <!-- CASTER WHEEL LINK -->
+    <joint name="caster_wheel_joint" type="fixed">
+        <parent link="chassis"/>
+        <child link="caster_wheel"/>
+        <origin xyz="${caster_wheel_offset_x} 0 ${caster_wheel_offset_z}"/>
     </joint>
-    <link name="front_right_wheel">
+    <link name="caster_wheel">
         <visual>
             <geometry>
-                <cylinder radius="${wheel_radius}" length="${wheel_thickness}"/>
+                <sphere radius="${caster_wheel_radius}"/>
             </geometry>
-            <material name="blue"/>
+            <material name="white"/>
         </visual>
         <collision>
             <geometry>
-                <sphere radius="${wheel_radius}"/>
+                <sphere radius="${caster_wheel_radius}"/>
             </geometry>
         </collision>
-        <xacro:inertial_cylinder mass="${wheel_mass}" length="${wheel_thickness}" radius="${wheel_radius}">
+        <xacro:inertial_sphere mass="${caster_wheel_mass}" radius="${caster_wheel_radius}">
             <origin xyz="0 0 0" rpy="0 0 0"/>
-        </xacro:inertial_cylinder>
+        </xacro:inertial_sphere>
     </link>
-    <!-- REAR RIGHT WHEEL (M4) -->
-    <joint name="rear_right_wheel_joint" type="continuous">
-        <parent link="base_link"/>
-        <child link="rear_right_wheel"/>
-        <origin xyz="${-wheel_offset_x} ${-wheel_offset_y} 0" rpy="${pi/2} 0 0" />
-        <axis xyz="0 0 -1"/>
-    </joint>
-    <link name="rear_right_wheel">
-        <visual>
-            <geometry>
-                <cylinder radius="${wheel_radius}" length="${wheel_thickness}"/>
-            </geometry>
-            <material name="blue"/>
-        </visual>
-        <collision>
-            <geometry>
-                <sphere radius="${wheel_radius}"/>
-            </geometry>
-        </collision>
-        <xacro:inertial_cylinder mass="${wheel_mass}" length="${wheel_thickness}" radius="${wheel_radius}">
-            <origin xyz="0 0 0" rpy="0 0 0"/>
-        </xacro:inertial_cylinder>
-    </link>
-    <!-- ALIAS MID-WHEEL JOINTS FOR 2WD / DIFF-DRIVE COMPATIBILITY -->
-    <joint name="left_wheel_joint" type="continuous">
-        <parent link="base_link"/>
-        <child link="left_wheel"/>
-        <origin xyz="0 ${wheel_offset_y} 0" rpy="-${pi/2} 0 0" />
-        <axis xyz="0 0 1"/>
-    </joint>
-    <link name="left_wheel"/>
-    <joint name="right_wheel_joint" type="continuous">
-        <parent link="base_link"/>
-        <child link="right_wheel"/>
-        <origin xyz="0 ${-wheel_offset_y} 0" rpy="${pi/2} 0 0" />
-        <axis xyz="0 0 -1"/>
-    </joint>
-    <link name="right_wheel"/>
+    <gazebo reference="caster_wheel">
+        <mu1 value="0.001"/>
+        <mu2 value="0.001"/>
+    </gazebo>
 </robot>

Commit message: feat: add robot description, lidar sensor, and ROS2 configuration files

File: robot/description/lidar.xacro (robot description, xacro)
@@ -1,8 +1,11 @@
 <?xml version="1.0"?>
 <robot xmlns:xacro="http://www.ros.org/wiki/xacro" >
+    <!-- base_link là tâm xoay của xe (tâm 4 bánh skid-steer); odometry quay
+         quanh điểm này. Đo thực tế: tâm LiDAR nằm trước tâm 4 bánh ~8 cm.
+         Gắn thẳng vào base_link để offset này không phụ thuộc hình chassis. -->
     <joint name="laser_joint" type="fixed">
-        <parent link="chassis"/>
+        <parent link="base_link"/>
         <child link="laser_frame"/>
-        <origin xyz="0.122 0 0.212" rpy="0 0 0"/>
+        <origin xyz="0.08 0 0.202" rpy="0 0 0"/>
     </joint>
     <link name="laser_frame">

File: robot/description/robot.urdf (robot description, URDF)
Before this commit: robot robot, 10 links, 9 joints
Joints:
- joint laser_joint: origin xyz=0.122 0 0.212 rpy=0 0 0 -> xyz=0.08 0 0.202 rpy=0 0 0; parent chassis -> base_link
